File: Host-50pin/Pi-Flex_15pin_150mm/capablerobot_CRAJEA_Pi-Flex_15pin_150mm.kicad_pcb (KiCad board)
At the start: 2 copper layers, 25.5 x 150 mm, 7 parts, among them J1 WE_686715100001_FLEX, J2 WE_687650100002_FLEX, Q1 BSS138APW, Q2 BSS138APW

Commit message: Change silk text
Other:
- board text added: "Capable Robot Components PI Flex, 15pin 150mm opposite side contacts [CRAJEA]"
- board text removed: "Capable Robot Components PI Flex, 15pin 150mm opposite side contacts Rev. 1.0.0"
