File: Host-50pin/Dual-Pi-Flex_22pin_150mm_24mm/capablerobot_CR8GPC_Dual-Pi-Flex_150mm_24mm.kicad_pcb (KiCad board)
At the start: 2 copper layers, 35.5 x 150 mm, 13 parts, among them Q1 BSS138APW, Q2 BSS138APW

Commit message: Update silk text
Parts:
- AntMicro MIPI Host: renamed from ANTMICRO MIPI HOST
